File: schematics/clock/change.kicad_sch (KiCad schematic)
At the start: 0 parts

Commit message: add change mode case
Parts:
- added C5: 0.01u, symbol Device:C
- added R6, R7: 1K, symbol Device:R
- added SW2: SW_SPDT, symbol Switch:SW_SPDT
- added U6: LM555xM, Package_SO:SOIC-8_3.9x4.9mm_P1.27mm, symbol breadboard:LM555xM
Connections:
- new net: R6.2, SW2.3 (C), U6.4 (~{RST})
- new net: R7.2, SW2.1 (A), U6.2 (TRIG)
- new net: C5.1, U6.5 (CONT)
- new net +5V: R6.1, R7.1, U6.7 (DISCH), U6.8 (VCC)
- new net GND: C5.2, SW2.2 (B), U6.1 (GND), U6.6 (THRES)
- new net clock_step: U6.3 (OUT)
