File: schematics/clock/register_A.kicad_sch (KiCad schematic)
At the start: 0 parts

Commit message: add register a
Parts:
- added D2, D3, D4, D5, D6, D7, D8, D9: LED, symbol Device:LED
- added RLED1, RLED2, RLED3, RLED4, RLED5, RLED6, RLED7, RLED8: 469, symbol Device:R
- added U7, U8: 74LS173, symbol 74xx:74LS173
- added U9: 74LS245, symbol 74xx:74LS245
Connections:
- new net: D2.2 (A), U7.3 (Q0), U9.2 (A0)
- new net: D3.2 (A), U7.4 (Q1), U9.3 (A1)
- new net: D4.2 (A), U7.5 (Q2), U9.4 (A2)
- new net: D5.2 (A), U7.6 (Q3), U9.5 (A3)
- new net: D2.1 (K), RLED1.1
- new net: D9.1 (K), RLED8.1
- new net: D6.1 (K), RLED5.1
- new net: D4.1 (K), RLED3.1
- new net: D8.1 (K), RLED7.1
- new net: D8.2 (A), U8.5 (Q2), U9.8 (A6)
- new net: D7.1 (K), RLED6.1
- new net: D7.2 (A), U8.4 (Q1), U9.7 (A5)
- new net: D5.1 (K), RLED4.1
- new net: D3.1 (K), RLED2.1
- new net: D6.2 (A), U8.3 (Q0), U9.6 (A4)
- new net: D9.2 (A), U8.6 (Q3), U9.9 (A7)
- new net +5V: U7.16 (VCC), U8.16 (VCC), U9.1 (A->B), U9.20 (VCC)
- new net CLK: U7.7 (Cp), U8.7 (Cp)
- new net CLR: U7.15 (Mr), U8.15 (Mr)
- new net GND: RLED1.2, RLED2.2, RLED3.2, RLED4.2, RLED5.2, RLED6.2, RLED7.2, RLED8.2, U7.1 (Oe1), U7.2 (Oe2), U7.8 (GND), U8.1 (Oe1), U8.2 (Oe2), U8.8 (GND), U9.10 (GND)
- new net ~{ENABLE}: U9.19 (CE)
- new net ~{LOAD}: U7.10 (E2), U7.9 (E1), U8.10 (E2), U8.9 (E1)
Other:
- note added: "data enable"
- note added: "low B->A ; high A->B"
- note added: "output control always on for led"
- note added: "output enable low-> all channels active high-> all channels disabled (high impedance)"
